File: pcb/gpsdo.sch (KiCad schematic (older format))
At the start: 71 parts

Commit message: PCB progress
Parts:
- added C? (x2): 100n, symbol Device:C
- added C? (x2): 10u, symbol Device:C
- added J?: 12V, symbol Connector:Jack-DC
- added R?: 200K, symbol Device:R
- added R?: 1K, symbol Device:R
- R? (x2): value 680 -> 7K5
- R? (x2): value 330 -> 3K
Connections:
- net SDI is gone; now on net SPI_SDI: IC?.13 (13_SDI), M?.32 (P0.20)
- net SDO is gone; now on net SPI_SDO: IC?.12 (12_SDO), M?.30 (P0.17)
- net +10V: now also C?.2, C?.2; no longer Y?.4 (Us)
- net +12V: now also Y?.4 (Us), J?.1
- net +3V3: now also C?.2, C?.2
- net EN_10V: now also M?.41 (NFC1/P0.09)
- net EN_1V2: now also M?.43 (NFC2/P0.10)
- net FPGA_INT: now also M?.20 (P0.12); no longer M?.12 (P0.26)
- net GND: now also C?.1, C?.1, C?.1, C?.1, J?.2, R?.2, R?.2
- net SCL: now also M?.15 (AIN3/P0.05); no longer M?.17 (P1.09)
- net SDA: now also M?.14 (P0.06); no longer M?.15 (AIN3/P0.05)
- net ~UC_RESET: now also U?.27 (PGOOD)
- net ~DAC_ALERT: now reaches U?.1 (~ALERT)
- net ~DAC_ALERT: now also M?.4 (AIN4/P0.28)
- net SPI_SDO: now reaches U?.10 (SDO)
- net ~DAC_LOAD: now reaches U?.11 (~LDAC)
- net ~DAC_LOAD: now also M?.9 (AIN7/P0.31)
- net SPI_SDI: now reaches U?.12 (SDI)
- net ~DAC_CS: now reaches U?.13 (~SYNC)
- net ~DAC_CS: now also M?.12 (P0.26)
- net SPI_CLK: now reaches U?.14 (SCLK)
- net SPI_CLK: now also IC?.15 (15_SCK), M?.34 (P0.22)
- net ~DAC_CLEAR: now reaches U?.2 (~CLEAR)
- net ~DAC_CLEAR: now also M?.8 (AIN5/P0.29)
- net ~DAC_RESET: now reaches U?.3 (~RESET)
- net ~DAC_RESET: now also M?.10 (AIN6/P0.30)
- net at U?.25 (F_PWM): now also R?.1
- net at U?.6 (ROSC): now also R?.1
- net FPGA_SS renamed ~FPGA_CS
- net ~FPGA_CS: now also M?.35 (P0.24); no longer M?.34 (P0.22)
- net OCXO_10MHZ renamed OCXO_OUTPUT
- removed net SCK: IC?.15 (15_SCK), M?.35 (P0.24)
- no-connect marks 16 -> 17
Other:
- note removed: "PGOOD:\nRESET tree?"
- note removed: "best practices,\nmax load?"
- note removed: "caps?"
- note removed: "control"
- note removed: "interrupt"
- moved on the sheet: C?, J?, R?, U?, Y?

Commit message: schematic progress
Parts:
- added C22, C23: 1u, symbol Device:C
- added C27, C30, C31, C32: 10n, symbol Device:C
- added D3: D, symbol Device:D
- added R18: 470, symbol Device:R
- added R19, R20, R21: 1K, symbol Device:R
- added SW1: MCML4-112B, symbol Switch:SW_Push_LED
- added SW2, SW3: MCML4-112W, symbol Switch:SW_Push_LED
- added SW4: MCML4-112R, symbol Switch:SW_Push_LED
- added U3: MIC5365-1.2YC5, Package_TO_SOT_SMD:SOT-353_SC-70-5, symbol Regulator_Linear:MIC5365-3.3YC5
- C38: renamed from C?; value 1n -> 100p
- C41: renamed from C?; value C -> 100n
- J5: renamed from J?; value 12V -> 13-16V DC
- gave numbers to parts that had none: 75
Connections:
- net SWCLK is gone; now on net SWDCLK: J1.4 (Pin_4)
- net +10V: now also C20.1, L2.1, R12.1, R15.2; no longer C21.1, L3.1, R13.1, R16.2
- net +12V: now also C21.1, L3.1, R13.1, R16.2; no longer J5.1, U1.13 (VIN1), U1.18 (VIN2), U1.38 (VIN3)
- net +1V2: now also C23.1, U3.5 (VOUT); no longer C20.1, L2.1, R12.1, R15.2
- net +3V3: now also C22.1, U3.1 (VIN)
- net EN_10V: now also U1.20 (EN2); no longer U1.40 (EN3)
- net EN_1V2: now also M1.16 (P0.08), U3.3 (EN); no longer M1.43 (NFC2/P0.10), U1.20 (EN2)
- net GND: now also C22.2, C23.2, C27.2, C30.2, C31.2, C32.2, SW1.1, SW1.3 (K), SW2.1, SW2.3 (K), SW3.1, SW3.3 (K), SW4.1, SW4.3 (K), U3.2 (GND)
- net BTN_BLU: now reaches IC1.22
- net BTN_BLU: now also C27.1, SW1.2
- net LED_BLU: now reaches IC1.23
- net LED_BLU: now also R18.1
- net BTN_WHT1: now reaches IC1.26
- net BTN_WHT1: now also C30.1, SW2.2
- net LED_WHT1: now reaches IC1.27
- net LED_WHT1: now also R19.1
- net BTN_WHT2: now reaches IC1.29 (29_GBIN)
- net BTN_WHT2: now also C31.1, SW3.2
- net LED_WHT2: now reaches IC1.30 (30_GBIN)
- net LED_WHT2: now also R20.1
- net BTN_RED: now reaches IC1.31
- net BTN_RED: now also C32.1, SW4.2
- net LED_RED: now reaches IC1.32
- net LED_RED: now also R21.1
- new net: D3.2 (A), J5.1
- new net: R18.2, SW1.4 (A)
- new net: R20.2, SW3.4 (A)
- new net: R21.2, SW4.4 (A)
- new net: R19.2, SW2.4 (A)
- new net +15V: D3.1 (K), U1.13 (VIN1), U1.18 (VIN2), U1.38 (VIN3)
- new net EN_12V: M1.43 (NFC2/P0.10), U1.40 (EN3)
- no-connect marks 17 -> 27
Other:
- note added: "close to FPGA"
- note removed: "buttons\nLEDs\n"
- moved on the sheet: C1, C10, C14, C15, C16, C17, C18, C19, C2, C20, C21, C3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

Commit message: schematic progress
Parts:
- removed R14: R, symbol Device:R
- removed Y1: 32786Hz, symbol Device:Crystal
- added R17: 2K2, symbol Device:R
- added R18, R20: 600, symbol Device:R
- added R19: 160, symbol Device:R
- added R21: 200, symbol Device:R
- added R22: 18, symbol Device:R
- added R23: 57, symbol Device:R
- added Y1: 32768, symbol Device:Crystal_Small
- C5: renamed from C6; value C -> 10n
- C7: renamed from C8; value C -> 10n
- C9: renamed from C10; value C -> 10n
- R11, R12, R13: value R -> 20K
- R15: value R -> 12K
- R16: value R -> 3K3
- renumbered C2 to C1, C1 to C10, C15 to C14, C16 to C15, C17 to C16, C14 to C17, C22 to C19, C3 to C2, C19 to C20, C20 to C21, C21 to C22, C4 to C3, C5 to C4, C7 to C6, C9 to C8, R17 to R14, R6 to R2, R18 to R24, R19 to R25, R20 to R26, R21 to R27, R22 to R28, R23 to R29, R2 to R3, R24 to R30, R25 to R31, R26 to R32, R7 to R4, R3 to R5, R8 to R6, R4 to R7, R5 to R8, U2 to U1, U1 to U2
Connections:
- net +10V: now also R16.2; no longer R15.2
- net +12V: now also R17.2; no longer R16.2
- net +3V3: now also R15.2
- net GND: now also R21.1, R22.1, R23.1; no longer R15.1, R16.1
- net at C12.2, M1.11 (XL1/P0.00): now also Y1.2
- net at C13.2, M1.13 (XL2/P0.01): now also Y1.1
- new net: R17.1, R20.2
- new net: R20.1, R23.2
- new net: R15.1, R18.2
- new net: R18.1, R21.2
- new net: R16.1, R19.2
- new net: R19.1, R22.2
Other:
- moved on the sheet: C1, C10, C11, C12, C13, C14, C15, C16, C17, C18, C19, C2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

Commit message: schematic progress
Parts:
- added U6: 74LVC1G17, symbol 74xGxx:74LVC1G17
- C11: value C -> 100n
- D3: value D -> S3M
- J5: value 13-16V DC -> 14-16V DC
- renumbered C24 to C23, C23 to C24, C28 to C27, C29 to C28, C27 to C29, C37 to C36, C36 to C37, U6 to U7
Connections:
- net PLL_OUT_10MHZ is gone; now on net PLL_OUT_REF: U4.13 (CLK0)
- net +3V3: now also U6.5 (VCC)
- net GND: now also U6.3 (GND)
- net PLL_OUT_REF: now also U6.2; no longer IC1.6 (6_GBIN), U4.15 (CLK7)
- net GPS_1PPS renamed GPS_PULSE
- net PLL_OUT1 renamed PLL_OUT_1
- net PLL_OUT2 renamed PLL_OUT_2
- net PLL_OUT3 renamed PLL_OUT_3
- net PLL_OUT4 renamed PLL_OUT_4
- net PLL_OUT5 renamed PLL_OUT_5
- net PLL_OUT6 renamed PLL_OUT_6
- new net PLL_OUT_7: U4.15 (CLK7)
- new net REF_DIGITAL: IC1.6 (6_GBIN), U6.4
Other:
- note added: "startup:\n 600mA\naverage:\n 250mA"
- note removed: "3.3V MAX INPUT"
- note removed: "Schmidt Trigger?"
- note removed: "output\nvoltage?"
- moved on the sheet: C19, C23, C24, C25, C26, C27, C28, C33, C36, R14, U3, U4
