File: pcb/gpsdo.sch (KiCad schematic (older format))
At the start: 101 parts, among them IC1 ICE40LP384-SG32, J1 JTAG, J2 USB_B_Micro, J3 USB_B_Micro, J4 Display SSD1306, J5 14-16V DC, J6 Conn_Coaxial, M1 E73-2G4M08S1C-52840, SW1 MCML4-112B, SW2 MCML4-112W, SW3 MCML4-112W, SW4 MCML4-112R, U1 Si7020-A20, U2 TPS652510, U3 MIC5365-1.2YC5, U4 Si5351C-B-GM, U5 uBlox NEO-7M, U6 74LVC1G17, U7 AD5761R, Y1 32768, Y2 8663-XS

Commit message: UI: rotary encoder would be nice, cleanup
Parts:
- removed C30, C31: 10n, symbol Device:C
- removed R25, R26: 1K, symbol Device:R
- removed SW2, SW3: MCML4-112W, symbol Switch:SW_Push_LED
- added C? (x3): 10n, symbol Device:C
- added D?: GREEN, symbol Device:LED
- added R?: 1K, symbol Device:R
- added SW?: EC11, symbol Device:Rotary_Encoder_Switch
- C29, C32: value 10n -> 100n
- J4: value Display SSD1306 -> SSD1306
Connections:
- net labels added: ENCODER_A, ENCODER_B, ENCODER_BTN, LED_GRN
- net labels removed: BTN_WHT1, BTN_WHT2, LED_WHT1, LED_WHT2
- wire segments 482 -> 474
Other:
- note added: "BIAS?"
- note added: "REAR PANEL"
- note removed: "replace with\nmultiple\nADT7410?"
- moved on the sheet: C11, C12, C13, C23, C25, C26, C27, C28, C29, C32, D1, D2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

Commit message: remove some errors and warnings
Parts:
- gave numbers to parts that had none: 6
- renumbered C12 to C11, C13 to C12, C11 to C13, C23 to C18, C25 to C19, C18 to C20, C26 to C21, C27 to C22, C19 to C23, C28 to C24, C20 to C26, C21 to C27, C22 to C28, C24 to C30, C29 to C32, C32 to C33, C33 to C34, C34 to C35, C35 to C36, C36 to C37, C37 to C38, C38 to C39, C39 to C40, C40 to C41, C41 to C42, D2 to D3, D3 to D4, D4 to D5, J4 to J2, J6 to J3, J2 to J4, J3 to J6, R18 to R19, R19 to R20, R20 to R21, R21 to R22, R22 to R23, R23 to R24, R24 to R25, R27 to R26, R28 to R27, R29 to R28, R30 to R29, R31 to R30, R32 to R31, SW1 to SW2, SW4 to SW3, U6 to U3, U3 to U4, U4 to U5, U5 to U6
Connections:
- wire segments 474 -> 477
Other:
- moved on the sheet: D4, D5, J5

Commit message: power concepts; bias and digitze OCXO output
Parts:
- added C22: 10u, symbol Device:C
- added R18, R19: 10K, symbol Device:R
- R11, R12, R13: value 20K -> 40K
- R16: value 3K3 -> 3K
- R21: renamed from R19; value 600 -> 680
- R22: renamed from R20; value 160 -> 470
- R24: renamed from R22; value 200 -> 120
- R25: renamed from R23; value 18 -> 8
- renumbered C22 to C24, C24 to C25, C25 to C26, C26 to C27, C27 to C28, C28 to C29, C29 to C30, C30 to C31, C31 to C32, C32 to C33, C33 to C34, C34 to C35, C35 to C36, C36 to C37, C37 to C39, C39 to C40, C40 to C41, C41 to C42, C42 to C43, R18 to R20, R21 to R23, R24 to R26, R25 to R27, R26 to R28, R27 to R29, R28 to R30, R29 to R31, R30 to R32, R31 to R33
Connections:
- net labels added: OCXO_DIGITAL
- net labels removed: REF_DIGITAL
- wire segments 477 -> 485
Other:
- note added: "Output stages\nwith buffers?"
- note added: "dummy load\nfor 10V rail?"
- note removed: "BIAS?"
- note removed: "Output\nstages"
- moved on the sheet: C18, C19, C21, C24, C25, C35, C36, C37, C39, C40, R14, R30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

Commit message: power progress, cleanup
Parts:
- removed C23, C31: 1u, symbol Device:C
- removed C28, C29: C, symbol Device:C
- removed C39: 10u, symbol Device:C
- removed R11, R12: 40K, symbol Device:R
- removed R22: 470, symbol Device:R
- removed R24: 120, symbol Device:R
- removed U4: MIC5365-1.2YC5, Package_TO_SOT_SMD:SOT-353_SC-70-5, symbol Regulator_Linear:MIC5365-3.3YC5
- added C17, C27: 1u, symbol Device:C
- added C26: 4u7, symbol Device:C
- added C30: 10n, symbol Device:C
- added C32, C38: 10u, symbol Device:C
- added R18: 43K, symbol Device:R
- added R20, R26: 1K8, symbol Device:R
- added R27: 12K, symbol Device:R
- added R28, R29: 470, symbol Device:R
- added R30: 13, symbol Device:R
- added R7: 100K, symbol Device:R
- added U?: LT1763xS8, Package_SO:SO-8_3.9x4.9mm_P1.27mm, symbol linear_technology:LT1763xS8
- C1, C14, C15, C16, C2: value C -> 47n
- C11, C12: value C -> DNP
- C25: renamed from C27; value C -> 10u
- C3: value C -> 10u
- C4: value C -> 12p
- C5, C7, C9: value 10n -> 4n7
- C6: value C -> 82p
- C8: value C -> 22p
- L1, L2, L3: value L -> 4u7
- R1: value R -> 12K
- R13: value 40K -> 43K
- R14: renamed from R23; value 600 -> 3K
- R15: value 12K -> 43K
- R16: value 3K -> 12K
- R17: value 2K2 -> 43K
- R19: renamed from R26; value 57 -> 82
- R2: value R -> 100K
- R21: value 680 -> 43K
- R25: value 8 -> 0
- R3: value R -> 7K5
- R4, R6: value R -> 300K
- R5: value R -> 4K7
- R8: renamed from R7; value 200K -> 100K
- renumbered C17 to C18, C18 to C19, C19 to C20, C20 to C21, C21 to C22, C22 to C23, C25 to C28, C26 to C29, C30 to C31, C32 to C33, C33 to C34, C34 to C35, C35 to C36, C36 to C37, C37 to C39, C38 to C40, C40 to C41, C41 to C42, C42 to C43, C43 to C44, R9 to R10, R10 to R11, R14 to R12, R18 to R22, R19 to R23, R20 to R24, R27 to R31, R28 to R32, R29 to R33, R30 to R34, R31 to R35, R32 to R36, R33 to R37, R8 to R9, U3 to U4
Connections:
- net labels added: PGOOD
- wire segments 485 -> 521
- no-connect marks 27 -> 26
Other:
- note added: "Compensation components,\nsee datasheet => Loop Compensation\n\nf_switch = 900 KHz\nf_c := f_switch/10=90 KHz\ng_M = 130 u/Ohm\ngm_ps = 10 A/V\nrc := 2*pi * f_c * co / (g_M * gm_ps)\ncc := rl * co / rc\ncroll := Resr * co / rc\nResr = 0.1Ohm\nfp_roll := 1/(2*pi * rc * croll)\n? fp_roll >= 2*f_c"
- note added: "close to DAC"
- note added: "i1 = 250mA average, 500mA max\nrl1 := 40Ohm\nco1 = 14uF\nrc1 := 13533Ohm => 12KOhm\ncc1 := 46nF => 47nF\ncroll1 := 12pF => 12pF\nfp_roll1 := 1.10MHz [OK]\n\ni2 = 50mA?\nrl2 := 60Ohm\nco2 = 7uF\nrc2 := 6766Ohm => 7K5Ohm\ncc2 := 56nF => 47nF\ncroll2 := 93pF => 82pF\nfp_roll2 := 259KHz [OK]\n\ni3 = 50uA\nrl3 := 40kOhm\nco3 = 1.1uF\nrc3 := 1063Ohm => 4K7Ohm\ncc3 := 10uF => 10uF\ncroll3 := 23pF => 22p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"
- note removed: "close to FPGA"
- note removed: "dummy load\nfor 10V rail?"
- note removed: "startup:\n 600mA\naverage:\n 250mA"
- moved on the sheet: C10, C25, J3, L1, R14, R19, U6

Commit message: LEDs, front/rear panel
Parts:
- added C22: 100n, symbol Device:C
- added D3: WHITE, symbol Device:LED
- added J10: CLK4, symbol Connector:Conn_Coaxial
- added J12: CLK3, symbol Connector:Conn_Coaxial
- added J13: CLK2, symbol Connector:Conn_Coaxial
- added J14: CLK1, symbol Connector:Conn_Coaxial
- added J15: CLK0, symbol Connector:Conn_Coaxial
- added J2: EXT_CLOCK, symbol Connector:Conn_Coaxial
- added J5: CLK7, symbol Connector:Conn_Coaxial
- added J7: CLK6, symbol Connector:Conn_Coaxial
- added J9: CLK5, symbol Connector:Conn_Coaxial
- added R24: 1K, symbol Device:R
- added U6: 74LVC1G17, symbol 74xGxx:74LVC1G17
- J8: renamed from J3; value Conn_Coaxial -> GPS_ANT
- gave numbers to parts that had none: 1
- renumbered C21 to C19, C19 to C20, C20 to C21, C22 to C23, C25 to C24, C26 to C25, C27 to C26, C24 to C27, C23 to C31, C31 to C32, C32 to C33, C33 to C34, C34 to C35, C35 to C36, C38 to C37, C36 to C38, C37 to C39, C39 to C40, C40 to C41, C41 to C42, C42 to C43, C43 to C44, C44 to C45, D3 to D4, D4 to D5, D5 to D6, J6 to J11, J2 to J3, J5 to J6, R13 to R12, R14 to R13, R15 to R14, R16 to R15, R17 to R16, R18 to R17, R12 to R18, R24 to R22, R25 to R23, R26 to R25, R22 to R26, R23 to R27, R27 to R28, R28 to R29, R29 to R30, R30 to R31, R31 to R32, R32 to R33, R33 to R34, R34 to R35, R35 to R36, R36 to R37, R37 to R38, U5 to U4, U4 to U5, U6 to U7, U7 to U8
Connections:
- net +3V3: now also U6.5 (VCC)
- net ENCODER_A: now also IC1.23; no longer IC1.22
- net ENCODER_B: now also IC1.26; no longer IC1.23
- net ENCODER_BTN: now also IC1.27; no longer IC1.26
- net GND: now also J10.2 (Ext), J12.2 (Ext), J13.2 (Ext), J14.2 (Ext), J15.2 (Ext), J2.2 (Ext), J5.2 (Ext), J7.2 (Ext), J9.2 (Ext), R24.2, U6.3 (GND)
- net GPS_PULSE: now also IC1.19 (19_GBIN); no longer IC1.20 (20_GBIN)
- net LED_GRN: now also IC1.20 (20_GBIN); no longer IC1.27
- net PLL_OUT_REF: now also U6.2
- net at U4.1 (XA): now also C22.1
- net PLL_OUT_1 renamed CLKOUT_1
- net CLKOUT_1: now also J14.1 (In)
- net PLL_OUT_2 renamed CLKOUT_2
- net CLKOUT_2: now also J13.1 (In)
- net PLL_OUT_3 renamed CLKOUT_3
- net CLKOUT_3: now also J12.1 (In)
- net PLL_OUT_4 renamed CLKOUT_4
- net CLKOUT_4: now also J10.1 (In)
- net PLL_OUT_5 renamed CLKOUT_5
- net CLKOUT_5: now also J9.1 (In)
- net PLL_OUT_6 renamed CLKOUT_6
- net CLKOUT_6: now also J7.1 (In)
- net PLL_OUT_7 renamed CLKOUT_7
- net CLKOUT_7: now also J5.1 (In)
- new net: C22.2, J2.1 (In)
- new net: D3.1 (K), R24.1
- new net CLKOUT_0: J15.1 (In), U6.4
- new net LED_WHT: D3.2 (A), IC1.22
- no-connect marks 26 -> 24
Other:
- note added: "check output voltage PP\nof 0-3.3V vs requirement\nof equipment. 1Vpp?"
- note removed: "Output stages\nwith buffers?"
- moved on the sheet: C20, C21, C23, C27, C28, C29, C31, C32, C34, C35, C36, C37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

Commit message: stub verilog implementation to see how much logic fits into the LP384 ; schematic adaptions for that
Parts:
- removed C35: 100n, symbol Device:C
- removed D2: GREEN, symbol Device:LED
- removed D3: WHITE, symbol Device:LED
- removed R22, R24: 1K, symbol Device:R
- removed R32: 470, symbol Device:R
- removed SW2: MCML4-112B, symbol Switch:SW_Push_LED
Connections:
- net LED_GRN is gone; now on net ENCODER_A: IC1.20 (20_GBIN)
- net LED_WHT is gone; now on net ENCODER_B: IC1.22
- net BTN_RED: now also IC1.26; no longer IC1.31
- net ENCODER_A: no longer IC1.23
- net ENCODER_B: no longer IC1.26
- net ENCODER_BTN: now also IC1.23; no longer IC1.27
- net LED_RED: no longer IC1.32
- net BTN_BLU renamed DISPLAY2
- net LED_BLU renamed DISPLAY3
- new net DISPLAY1: IC1.27
- new net DISPLAY4: IC1.31
- no-connect marks 24 -> 25
Other:
- moved on the sheet: J10, J12, J13, J14, J15, J5, J7, J9, U6

Commit message: FPGA progress, interface and schematic-cleanup
Parts:
- removed R33: 1K, symbol Device:R
- added AE?: ANT, symbol Device:Antenna
- added D?: OUT3, symbol Device:LED
- added D?: OUT6, symbol Device:LED
- added D?: GREEN, symbol Device:LED
- added D?: OUT0, symbol Device:LED
- added D?: OUT7, symbol Device:LED
- added D? (x2): RED, symbol Device:LED
- added D?: OUT4, symbol Device:LED
- added D?: OUT1, symbol Device:LED
- added D?: WHITE, symbol Device:LED
- added D?: OUT5, symbol Device:LED
- added D?: OUT2, symbol Device:LED
- added JP?: ANT_SEL, symbol Jumper:Jumper_3_Bridged12
- added R?: 50, symbol Device:R
- added R? (x4): 680, symbol Device:R
- added R?: 470, symbol Device:R
- J8: value GPS_ANT -> EXT_ANT
- SW3: value MCML4-112R -> MCML4-112B
Connections:
- net DISPLAY3 is gone; now on net DISPLAY2: IC1.30 (30_GBIN)
- net DISPLAY4 is gone; now on net BLUE_HI: IC1.31
- net DISPLAY1: now also IC1.29 (29_GBIN), D?.2 (A), D?.2 (A), D?.2 (A), R?.1; no longer IC1.27
- net DISPLAY2: now also D?.2 (A), D?.2 (A), D?.2 (A), R?.1; no longer IC1.29 (29_GBIN)
- net EN_10V: now also M1.16 (P0.08); no longer M1.41 (NFC1/P0.09)
- net EN_12V: now also M1.41 (NFC1/P0.09); no longer M1.43 (NFC2/P0.10)
- net EN_1V2: now also M1.22 (P0.07); no longer M1.16 (P0.08)
- net GND: now also R?.2, R?.2; no longer SW3.3 (K)
- net PLL_OUT_REF: now also R?.1
- net FPGA_WDT: now reaches IC1.8 (8_GBIN)
- net FPGA_WDT: now also M1.43 (NFC2/P0.10)
- net FAULT: now reaches M1.2 (P1.10)
- net FAULT: now also D?.2 (A)
- net at U7.11 (RF_IN): now also JP?.2 (C); no longer J8.1 (In)
- net BLUE_HI: now reaches SW3.4 (A)
- net BLUE_HI: now also D?.2 (A), D?.2 (A), R?.1
- net BTN_RED renamed BTN_BLUE
- new net: J8.1 (In), JP?.3 (B)
- new net: AE?.1 (A), JP?.1 (A)
- new net: D?.1 (K), D?.1 (K), D?.1 (K), R?.2 (x3)
- new net: D?.1 (K), R?.1
- new net BLUE_LO: D?.1 (K), D?.1 (K), R?.2, SW3.3 (K)
- new net DISPLAY0: D?.2 (A), D?.2 (A), D?.2 (A), IC1.27, R?.1
- no-connect marks 25 -> 22
Other:
- note added: "LEDs green unless specified.\nOUT0..OUT7 to be placed next\nto CLKOUT_0..CLKOUT_7 jacks.\n"
- note added: "check output voltage PP\nof 0-3.3V vs requirement\nof equipment. 1Vpp?\n\nCheck if sine or square\nis needed."
- note removed: "check output voltage PP\nof 0-3.3V vs requirement\nof equipment. 1Vpp?"
- moved on the sheet: C29, C32, C34, C36, J10, J11, J12, J13, J14, J15, J3, J4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

Commit message: schematic progress
Parts:
- removed C22: 100n, symbol Device:C
- added R10, R11: 50, symbol Device:R
- R12: renamed from R10; value 10K -> 4K7
- R13: renamed from R11; value 10K -> 4K7
- gave numbers to parts that had none: 20
- renumbered C31 to C22, C30 to C28, C28 to C29, C29 to C30, C32 to C31, C33 to C32, C34 to C33, C36 to C34, C37 to C35, C38 to C36, C39 to C37, C40 to C38, C41 to C39, C42 to C40, C43 to C41, C44 to C42, C45 to C43, D5 to D13, D6 to D16, D4 to D6, J15 to J10, J5 to J12, J7 to J13, J9 to J14, J10 to J15, J12 to J5, J13 to J7, J14 to J9, R12 to R14, R13 to R15, R14 to R16, R15 to R17, R16 to R18, R17 to R19, R18 to R20, R19 to R21, R20 to R22, R21 to R23, R26 to R24, R27 to R25, R23 to R27, R25 to R28, R28 to R29, R29 to R30, R30 to R31, R31 to R32, R34 to R38, R35 to R39, R36 to R40, R37 to R41, R38 to R42, SW3 to SW2, U5 to U4, U4 to U5
Connections:
- net EN_12V: now also M1.20 (P0.12); no longer M1.41 (NFC1/P0.09)
- net FPGA_INT: now also R10.1; no longer M1.20 (P0.12)
- net FPGA_WDT: now also R11.1; no longer M1.43 (NFC2/P0.10)
- net GPS_PULSE: now also M1.17 (P1.09)
- net at U5.1 (XA): now also J2.1 (In)
- net PLL_OUT_REF renamed PLL_INT_REF
- new net: M1.41 (NFC1/P0.09), R10.2
- new net: M1.43 (NFC2/P0.10), R11.2
- no-connect marks 22 -> 21
Other:
- note removed: "check output voltage PP\nof 0-3.3V vs requirement\nof equipment. 1Vpp?\n\nCheck if sine or square\nis needed."
- moved on the sheet: C20, C21, C22, C23, C27, C29, J2, R20, R24, R25, U4, U5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
