File: pcb/gpsdo.kicad_pcb (KiCad board)
At the start: 2 copper layers, 100 x 100 mm, 148 parts, among them IC1 ICE40LP384-SG32, J1 JTAG, J10 CLK0, J11 USB_B_Micro, J12 CLK7, J13 CLK6, J14 CLK5, J15 CLK4, J2 EXT_CLOCK, J3 SSD1306, J4 USB_B_Micro, J5 GPS_ANT, J6 CLK3, J7 Screw_Terminal_01x03, J8 CLK2, J9 CLK1, M1 E73-2G4M08S1C-52840, Q1 S9018, SW1 EC11, SW2 MCML4-112B, U1 Si7020-A20, U2 TPS652510, U3 LT1763xS8, U4 74LVC1G17, U5 Si5351C-B-GM, U6 74LVC1G17, U7 uBlox NEO-7M, U8 AD5761R, Y1 32768, Y2 8663-XS

Commit message: replace expensive Si7010 with two cheaper temp sensors
Parts:
- added C48: 100n, Capacitor_SMD:C_0402_1005Metric, F.Cu at (3.11, -152.0)
- added R49: 3K, Resistor_SMD:R_0603_1608Metric, F.Cu at (3.66, -154.2)
- added U9: AD5761R, Package_SO:TSSOP-16_4.4x5mm_P0.65mm, F.Cu at (-2.82, -152.1)
- C1: value 47n -> 100n
- C10: value 100n -> 4n7
- C12, C35: value DNP -> 100n
- C14: value 1u -> DNP; footprint Capacitor_SMD:C_0603_1608Metric -> Capacitor_SMD:C_0402_1005Metric
- C15: value 47n -> 1u; footprint Capacitor_SMD:C_0402_1005Metric -> Capacitor_SMD:C_0603_1608Metric
- C18: value 10u -> 47n; footprint Capacitor_SMD:C_0603_1608Metric -> Capacitor_SMD:C_0402_1005Metric
- C20: value 100n -> 10u; footprint Capacitor_SMD:C_0402_1005Metric -> Capacitor_SMD:C_0603_1608Metric
- C21, C23, C40: value 100n -> 10u; footprint Capacitor_SMD:C_0402_1005Metric -> Capacitor_SMD:C_1210_3225Metric
- C22: value 10u -> 100n; footprint Capacitor_SMD:C_1210_3225Metric -> Capacitor_SMD:C_0402_1005Metric
- C24: value 10u -> 4u7; footprint Capacitor_SMD:C_1210_3225Metric -> Capacitor_SMD:C_0603_1608Metric
- C25: value 4u7 -> 1u
- C26: value 1u -> 100n; footprint Capacitor_SMD:C_0603_1608Metric -> Capacitor_SMD:C_0402_1005Metric
- C3: value 10u -> 47n
- C31, C42: value 10n -> 100n
- C32: value 10u -> 10n; footprint Capacitor_SMD:C_0603_1608Metric -> Capacitor_SMD:C_0402_1005Metric
- C33: value 10n -> 10u; footprint Capacitor_SMD:C_0402_1005Metric -> Capacitor_SMD:C_0603_1608Metric
- C34: value 100n -> 10n
- C36: value 10u -> DNP; footprint Capacitor_SMD:C_1210_3225Metric -> Capacitor_SMD:C_0402_1005Metric
- C38: footprint Capacitor_SMD:C_0603_1608Metric -> Capacitor_SMD:C_1210_3225Metric
- C39: footprint Capacitor_SMD:C_1210_3225Metric -> Capacitor_SMD:C_0603_1608Metric
- C4: value 12p -> 10u
- C43: value 10p -> 10n
- C44: value 100n -> 10p
- C5: value 4n7 -> 12p
- C6: value 82p -> 4n7
- C7: value 4n7 -> 82p
- C8: value 22p -> 4n7
- C9: value 4n7 -> 22p
- J11: value USB_B_Micro -> CLK7; footprint dpiegdon:USB_Micro-B_Aliexpress_7.2mm_Pitch -> Connector_Coaxial:SMA_Molex_73251-1153_EdgeMount_Horizontal
- J12: value CLK7 -> USB_B_Micro; footprint Connector_Coaxial:SMA_Molex_73251-1153_EdgeMount_Horizontal -> dpiegdon:USB_Micro-B_Aliexpress_7.2mm_Pitch
- J2: value EXT_CLOCK -> SSD1306; footprint Connector_Coaxial:U.FL_Molex_MCRF_73412-0110_Vertical -> Connector_PinHeader_2.54mm:PinHeader_1x04_P2.54mm_Vertical
- J3: value SSD1306 -> EXT_CLOCK; footprint Connector_PinHeader_2.54mm:PinHeader_1x04_P2.54mm_Vertical -> Connector_Coaxial:U.FL_Molex_MCRF_73412-0110_Vertical
- J4: value USB_B_Micro -> GPS_ANT; footprint dpiegdon:USB_Micro-B_Aliexpress_7.2mm_Pitch -> Connector_Coaxial:U.FL_Molex_MCRF_73412-0110_Vertical
- J5: value GPS_ANT -> USB_B_Micro; footprint Connector_Coaxial:U.FL_Molex_MCRF_73412-0110_Vertical -> dpiegdon:USB_Micro-B_Aliexpress_7.2mm_Pitch
- R1: value 4K7 -> 12K; footprint Resistor_SMD:R_0603_1608Metric -> Resistor_SMD:R_0402_1005Metric
- R10: value 100K -> 10K
- R11: value 1K -> 50
- R13: value 50 -> 1K
- R15: value 1K -> 4K7; footprint Resistor_SMD:R_0402_1005Metric -> Resistor_SMD:R_0603_1608Metric
- R16: value 43K -> 10K
- R17: value 3K -> 43K
- R18: value 43K -> 3K; footprint Resistor_SMD:R_0402_1005Metric -> Resistor_SMD:R_0603_1608Metric
- R19: value 12K -> 43K
- R2: value 12K -> 100K
- R20: value 43K -> 12K
- R22: value 10K -> 43K
- R23: value 4K7 -> 10K
- R27: value 0 -> 4K7; footprint Resistor_SMD:R_0603_1608Metric -> Resistor_SMD:R_0402_1005Metric
- R3: value 100K -> 7K5
- R30: value 470 -> 0; footprint Resistor_SMD:R_0402_1005Metric -> Resistor_SMD:R_0603_1608Metric
- R31: value 1K8 -> 470; footprint Resistor_SMD:R_0603_1608Metric -> Resistor_SMD:R_0402_1005Metric
- R32: value 12K -> 1K8
- R33: value 470 -> 12K
- R35: value 13 -> 470
- R36: value 27 -> 13; footprint Resistor_SMD:R_0402_1005Metric -> Resistor_SMD:R_0603_1608Metric
- R38: value 680 -> 27
- R39: value DNP -> 680
- R4: value 7K5 -> 300K
- R40: value 680 -> DNP
- R43: value 50 -> 680
- R44: value 10K -> 50
- R45: value 7K5 -> 10K; footprint Resistor_SMD:R_0603_1608Metric -> Resistor_SMD:R_0402_1005Metric
- R46, R48: value 3K -> 7K5
- R47: value 7K5 -> 3K
- R5: value 300K -> 4K7
- R6: value 4K7 -> 300K
- R7: value 300K -> 100K
- R9: value 10K -> 1K; footprint Resistor_SMD:R_0603_1608Metric -> Resistor_SMD:R_0402_1005Metric
- U1: value Si7020-A20 -> MCP9808_MSOP; footprint Package_DFN_QFN:DFN-6-1EP_3x3mm_P1mm_EP1.5x2.4mm -> Package_SO:MSOP-8_3x3mm_P0.65mm
- U2: value TPS652510 -> MCP9808_MSOP; footprint Package_DFN_QFN:QFN-40-1EP_6x6mm_P0.5mm_EP4.6x4.6mm_ThermalVias -> Package_SO:MSOP-8_3x3mm_P0.65mm
- U3: value LT1763xS8 -> TPS652510; footprint Package_SO:SO-8_3.9x4.9mm_P1.27mm -> Package_DFN_QFN:QFN-40-1EP_6x6mm_P0.5mm_EP4.6x4.6mm_ThermalVias
- U4: value 74LVC1G17 -> LT1763xS8; footprint Package_TO_SOT_SMD:SOT-23-5 -> Package_SO:SO-8_3.9x4.9mm_P1.27mm
- U5: value Si5351C-B-GM -> 74LVC1G17; footprint Package_DFN_QFN:QFN-20-1EP_4x4mm_P0.5mm_EP2.7x2.7mm -> Package_TO_SOT_SMD:SOT-23-5
- U6: value 74LVC1G17 -> Si5351C-B-GM; footprint Package_TO_SOT_SMD:SOT-23-5 -> Package_DFN_QFN:QFN-20-1EP_4x4mm_P0.5mm_EP2.7x2.7mm
- U7: value uBlox NEO-7M -> 74LVC1G17; footprint RF_GPS:ublox_NEO -> Package_TO_SOT_SMD:SOT-23-5
- U8: value AD5761R -> uBlox NEO-7M; footprint Package_SO:TSSOP-16_4.4x5mm_P0.65mm -> RF_GPS:ublox_NEO
Connections:
- C1 pad 1: Net-(C1-Pad1) -> GND
- C1 pad 2: GND -> +3V3
- C10 pad 2: +3V3 -> Net-(C10-Pad2)
- C12 pad 2: Net-(C12-Pad2) -> +3V3
- C14 pad 2: +12V -> Net-(C14-Pad2)
- C15 pad 1: Net-(C15-Pad1) -> GND
- C15 pad 2: Net-(C15-Pad2) -> +12V
- C18 pad 1: GND -> Net-(C18-Pad1)
- C20 pad 1: +3V3 -> GND
- C20 pad 2: GND -> Net-(C20-Pad2)
- C21 pad 1: +3V3 -> Net-(C21-Pad1)
- C21 pad 2: GND -> /OCXO_OUTPUT
- C22 pad 1: Net-(C22-Pad1) -> +3V3
- C22 pad 2: /OCXO_OUTPUT -> GND
- C23 pad 1: +3V3 -> +12V
- C24 pad 1: +12V -> +3V3
- C25 pad 1: +3V3 -> +1V2
- C26 pad 1: +1V2 -> +3V3
- C31 pad 1: /ENCODER_B -> +3V3
- C32 pad 1: +10V -> /ENCODER_B
- C33 pad 1: /ENCODER_BTN -> +10V
- C34 pad 1: /BTN_BLUE -> /ENCODER_BTN
- C35 pad 1: Net-(C35-Pad1) -> /BTN_BLUE
- C36 pad 1: GND -> Net-(C36-Pad1)
- C36 pad 2: +15V -> GND
- C38 pad 2: +3V3 -> +15V
- C39 pad 2: +15V -> +3V3
- C4 pad 1: GND -> Net-(C4-Pad1)
- C4 pad 2: Net-(C4-Pad2) -> GND
- C40 pad 2: +3V3 -> +15V
- C41 pad 1: +3V3 -> GND
- C41 pad 2: GND -> +3V3
- C42 pad 1: Net-(C42-Pad1) -> +3V3
- C44 pad 1: +3V3 -> Net-(C44-Pad1)
- C45 pad 1: GND -> +3V3
- C45 pad 2: +10V -> GND
- C46 pad 1: +3V3 -> GND
- C46 pad 2: GND -> +10V
- C47 pad 1: +1V2 -> +3V3
- IC1 pad 32: (no net) -> /TEMP_ALERT
- J11 pad 1: /GPS_VBUS -> /CLKOUT_7
- J11 pad 2: /GPS_USB_D- -> GND
- J12 pad 1: /CLKOUT_7 -> /GPS_VBUS
- J12 pad 2: GND -> /GPS_USB_D-
- J2 pad 1: Net-(J2-Pad1) -> /SDA
- J2 pad 2: GND -> /SCL
- J3 pad 1: /SDA -> Net-(J3-Pad1)
- J3 pad 2: /SCL -> GND
- J4 pad 1: /UC_VBUS -> /GPS_EXT_RF
- J4 pad 2: /UC_USB_D- -> GND
- J5 pad 1: /GPS_EXT_RF -> /UC_VBUS
- J5 pad 2: GND -> /UC_USB_D-
- L1 pad 2: Net-(C15-Pad1) -> Net-(C16-Pad1)
- L2 pad 2: Net-(C16-Pad1) -> Net-(C17-Pad1)
- L3 pad 2: Net-(C17-Pad1) -> Net-(C18-Pad1)
- L4 pad 2: Net-(C35-Pad1) -> Net-(C36-Pad1)
- M1 pad 11: Net-(C12-Pad2) -> Net-(C13-Pad2)
- M1 pad 13: Net-(C13-Pad2) -> Net-(C14-Pad2)
- Q1 pad 3: /EN_10V_PU -> Net-(Q1-Pad3)
- R1 pad 1: Net-(Q1-Pad1) -> Net-(C5-Pad2)
- R1 pad 2: /~EN_10V -> Net-(C2-Pad1)
- R10 pad 1: Net-(R10-Pad1) -> +3V3
- R10 pad 2: Net-(R10-Pad2) -> /TEMP_ALERT
- R11 pad 1: Net-(R11-Pad1) -> /FPGA_INT
- R11 pad 2: GND -> Net-(M1-Pad41)
- R12 pad 1: /FPGA_INT -> /FPGA_WDT
- R12 pad 2: Net-(M1-Pad41) -> Net-(M1-Pad43)
- R13 pad 1: /FPGA_WDT -> +3V3
- R13 pad 2: Net-(M1-Pad43) -> /SCL
- R14 pad 2: /SCL -> /SDA
- R15 pad 1: +3V3 -> Net-(Q1-Pad1)
- R15 pad 2: /SDA -> /~EN_10V
- R16 pad 1: Net-(R16-Pad1) -> +12V
- R16 pad 2: +12V -> Net-(Q1-Pad3)
- R17 pad 2: Net-(R16-Pad1) -> +12V
- R18 pad 2: +3V3 -> Net-(R17-Pad1)
- R19 pad 2: Net-(R18-Pad1) -> +3V3
- R2 pad 1: Net-(C4-Pad2) -> Net-(R2-Pad1)
- R2 pad 2: Net-(C1-Pad1) -> GND
- R20 pad 2: +1V2 -> Net-(R19-Pad1)
- R21 pad 2: Net-(R20-Pad1) -> +1V2
- R22 pad 1: +3V3 -> Net-(R22-Pad1)
- R22 pad 2: /PGOOD -> Net-(R21-Pad1)
- R23 pad 2: /PLL_INT -> /PGOOD
- R24 pad 2: Net-(R17-Pad1) -> Net-(R18-Pad1)
- R25 pad 2: Net-(R19-Pad1) -> Net-(R20-Pad1)
- R26 pad 2: Net-(R21-Pad1) -> Net-(R22-Pad1)
- R27 pad 1: GND -> +3V3
- R27 pad 2: Net-(R27-Pad2) -> /PLL_INT
- R28 pad 2: Net-(C22-Pad1) -> Net-(C21-Pad1)
- R29 pad 1: Net-(C22-Pad1) -> Net-(C21-Pad1)
- R3 pad 1: Net-(R3-Pad1) -> Net-(C7-Pad2)
- R3 pad 2: GND -> Net-(C3-Pad1)
- R30 pad 1: Net-(D2-Pad1) -> GND
- R30 pad 2: GND -> Net-(R30-Pad2)
- R31 pad 1: Net-(R27-Pad2) -> Net-(D2-Pad1)
- R31 pad 2: Net-(R31-Pad2) -> GND
- R32 pad 1: +10V -> Net-(R30-Pad2)
- R33 pad 1: Net-(R33-Pad1) -> +10V
- R33 pad 2: Net-(R32-Pad2) -> Net-(R33-Pad2)
- R34 pad 2: Net-(R33-Pad1) -> Net-(R33-Pad2)
- R35 pad 1: Net-(R34-Pad1) -> Net-(R35-Pad1)
- R35 pad 2: Net-(R31-Pad2) -> Net-(R34-Pad1)
- R36 pad 1: Net-(R36-Pad1) -> Net-(R35-Pad1)
- R36 pad 2: /GPS_USB_D- -> Net-(R32-Pad2)
- R37 pad 2: /GPS_USB_D+ -> /GPS_USB_D-
- R38 pad 1: /DISPLAY0 -> Net-(R38-Pad1)
- R38 pad 2: Net-(D10-Pad1) -> /GPS_USB_D+
- R39 pad 1: Net-(C35-Pad1) -> /DISPLAY0
- R39 pad 2: Net-(JP1-Pad2) -> Net-(D10-Pad1)
- R4 pad 1: Net-(C6-Pad2) -> Net-(R4-Pad1)
- R4 pad 2: Net-(C2-Pad1) -> GND
- R40 pad 1: /DISPLAY1 -> Net-(C36-Pad1)
- R40 pad 2: Net-(D11-Pad1) -> Net-(JP1-Pad2)
- R41 pad 1: /DISPLAY2 -> /DISPLAY1
- R41 pad 2: /BLUE_LO -> Net-(D11-Pad1)
- R42 pad 1: /BLUE_HI -> /DISPLAY2
- R42 pad 2: Net-(D12-Pad1) -> /BLUE_LO
- R43 pad 1: /PLL_INT_REF -> /BLUE_HI
- R43 pad 2: GND -> Net-(D12-Pad1)
- R44 pad 1: +3V3 -> /PLL_INT_REF
- R44 pad 2: /CRESET_B -> GND
- R45 pad 1: Net-(R45-Pad1) -> +3V3
- R45 pad 2: /OCXO_VREF -> /CRESET_B
- R46 pad 1: /OCXO_VREF -> Net-(R46-Pad1)
- R46 pad 2: GND -> /OCXO_VREF
- R47 pad 1: Net-(C43-Pad1) -> /OCXO_VREF
- R47 pad 2: /DAC_VAL -> GND
- R48 pad 1: /DAC_VAL -> Net-(C44-Pad1)
- R48 pad 2: GND -> /DAC_VAL
- R5 pad 1: Net-(R5-Pad1) -> Net-(C9-Pad2)
- R5 pad 2: GND -> Net-(C4-Pad1)
- R6 pad 1: Net-(C8-Pad2) -> Net-(R6-Pad1)
- R6 pad 2: Net-(C3-Pad1) -> GND
- R8 pad 1: Net-(R10-Pad2) -> Net-(R8-Pad1)
- R8 pad 2: GND -> Net-(R7-Pad1)
- R9 pad 1: +12V -> Net-(R9-Pad1)
- R9 pad 2: /EN_10V_PU -> GND
- U1 pad 2: GND -> /SCL
- U1 pad 3: (no net) -> /TEMP_ALERT
- U1 pad 4: (no net) -> GND
- U1 pad 5: +3V3 -> GND
- U1 pad 6: /SCL -> GND
- U1 pad 7: (no net) -> GND
- U2 pad 1: Net-(R7-Pad1) -> /SDA
- U2 pad 2: Net-(C9-Pad2) -> /SCL
- U2 pad 3: Net-(C8-Pad2) -> /TEMP_ALERT
- U2 pad 4: Net-(R20-Pad1) -> GND
- U2 pad 6: Net-(R10-Pad1) -> GND
- U2 pad 7: Net-(R16-Pad1) -> +3V3
- U2 pad 8: Net-(C4-Pad2) -> +3V3
- U3 pad 1: +10V -> Net-(R6-Pad1)
- U3 pad 2: Net-(R31-Pad2) -> Net-(C10-Pad2)
- U3 pad 3: GND -> Net-(C9-Pad2)
- U3 pad 4: Net-(C28-Pad1) -> Net-(R21-Pad1)
- U3 pad 5: /EN_10V_PU -> GND
- U3 pad 6: GND -> Net-(R8-Pad1)
- U3 pad 7: GND -> Net-(R17-Pad1)
- U3 pad 8: +12V -> Net-(C5-Pad2)
- U4 pad 1: (no net) -> +10V
- U4 pad 2: Net-(C22-Pad1) -> Net-(R32-Pad2)
- U4 pad 4: /OCXO_DIGITAL -> Net-(C28-Pad1)
- U4 pad 5: +3V3 -> Net-(Q1-Pad3)
- U5 pad 1: Net-(J2-Pad1) -> (no net)
- U5 pad 2: (no net) -> Net-(C21-Pad1)
- U5 pad 3: /PLL_INT -> GND
- U5 pad 4: /SCL -> /OCXO_DIGITAL
- U5 pad 5: /SDA -> +3V3
- U6 pad 1: (no net) -> Net-(J3-Pad1)
- U6 pad 2: /PLL_INT_REF -> (no net)
- U6 pad 3: GND -> /PLL_INT
- U6 pad 4: /CLKOUT_0 -> /SCL
- U6 pad 5: +3V3 -> /SDA
- U7 pad 2: (no net) -> /PLL_INT_REF
- U7 pad 3: /GPS_PULSE -> GND
- U7 pad 4: (no net) -> /CLKOUT_0
- U7 pad 5: Net-(R36-Pad1) -> +3V3
- U8 pad 1: /~DAC_ALERT -> (no net)
- U8 pad 10: /SPI_SDO -> GND
- U8 pad 11: /~DAC_LOAD -> Net-(JP2-Pad2)
- U8 pad 12: /SPI_SDI -> GND
- U8 pad 13: /~DAC_CS -> GND
- U8 pad 14: /SPI_CLK -> (no net)
- U8 pad 15: +3V3 -> (no net)
- U8 pad 16: GND -> (no net)
- U8 pad 2: /~DAC_CLEAR -> (no net)
- U8 pad 3: /~DAC_RESET -> /GPS_PULSE
- U8 pad 4: Net-(C42-Pad1) -> (no net)
- U8 pad 5: GND -> Net-(R37-Pad1)
- U8 pad 6: GND -> Net-(R38-Pad1)
- U8 pad 7: Net-(C43-Pad1) -> +3V3
- U8 pad 8: +10V -> /~GPS_RESET
- U8 pad 9: (no net) -> /GPS_VCC_RF
- Y1 pad 1: Net-(C13-Pad2) -> Net-(C14-Pad2)
- Y1 pad 2: Net-(C12-Pad2) -> Net-(C13-Pad2)
- Y2 pad 2: Net-(C43-Pad1) -> Net-(C44-Pad1)
- Y2 pad 3: Net-(R45-Pad1) -> Net-(R46-Pad1)
Routing:
- net /GPS_VBUS: track 5.44 -> 0.00 mm, vias 1 -> 0
- net Net-(R36-Pad1): track 4.30 -> 0.00 mm
- net Net-(R35-Pad1): track 0.00 -> 4.30 mm
- net GND: track 33.4 -> 29.2 mm
- net /UC_VBUS: track 5.30 -> 2.46 mm
- net Net-(C35-Pad1): track 2.46 -> 0.00 mm
- net Net-(JP1-Pad2): track 1.91 -> 0.02 mm
- net /UC_USB_D+: track 5.16 -> 3.36 mm
- net +3V3: track 2.14 -> 1.11 mm, vias 1 -> 0
- net /GPS_USB_D-: track 7.32 -> 6.50 mm
- net /GPS_USB_D+: track 8.85 -> 8.03 mm
